File: SenseForge.kicad_sch (KiCad schematic)
At the start: 11 parts, among them J1 SHTC3, J2 PIR, J3 BH1750, J4 I2C, SW1 custom_button

Commit message: JLCPCB Part no. added
Parts:
- R1, R2: JLCPCB (none) -> C17414; Website (none) -> https://jlcpcb.com/partdetail/18102-0805W8F1002T5E/C17414
- R3, R4: JLCPCB (none) -> C17513; Website (none) -> https://jlcpcb.com/partdetail/18201-0805W8F1001T5E/C17513
Changed lines of the file:
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@@
+			)
+		)
+		(property "Website" "https://jlcpcb.com/partdetail/18102-0805W8F1002T5E/C17414"
+			(at 143.51 66.04 0)
+			(effects
+				(font
+					(size 1.27 1.27)
+				)
+				(hide yes)
+			)
+		)
+		(property "JLCPCB" "C17414"
+			(at 143.51 66.04 0)
+			(effects
+				(font
+					(size 1.27 1.27)
+				)
+				(hide yes)
 			)
 		)
@@
 			)
 		)
+		(property "Website" "https://jlcpcb.com/partdetail/18102-0805W8F1002T5E/C17414"
+			(at 133.35 66.04 0)
+			(effects
+				(font
+					(size 1.27 1.27)
+				)
+				(hide yes)
+			)
+		)
+		(property "JLCPCB" "C17414"
+			(at 133.35 66.04 0)
+			(effects
+				(font
+					(size 1.27 1.27)
+				)
+				(hide yes)
+			)
+		)
 		(pin "1"
 		)
@@
 			)
 		)
+		(property "Website" "https://jlcpcb.com/partdetail/18201-0805W8F1001T5E/C17513"
+			(at 85.09 100.33 0)
+			(effects
+				(font
+					(size 1.27 1.27)
+				)
+				(hide yes)
+			)
+		)
+		(property "JLCPCB" "C17513"
+			(at 85.09 100.33 0)
+			(effects
+				(font
+					(size 1.27 1.27)
+				)
+				(hide yes)
+			)
+		)
 		(pin "1"
 		)
@@
 			(at 68.58 86.36 0)
 			(effects
+				(font
+					(size 1.27 1.27)
+				)
+				(hide yes)
+			)
+		)
+		(property "Website" "https://jlcpcb.com/partdetail/18201-0805W8F1001T5E/C17513"
+			(at 68.58 86.36 0)
+			(effects
+				(font
+					(size 1.27 1.27)
+				)
+				(hide yes)
+			)
+		)
+		(property "JLCPCB" "C17513"
+			(at 68.58 86.36 0)
+			(effects

Commit message: update: latest SenseForge PCB and schematic changes
Parts:
- SW1: footprint Button_Switch_SMD:SW_Push_1P1T_NO_CK_KMR2 -> _myLibrary:button_push_sms; Field5 (none) -> https://asset.conrad.com/media10/add/160267/c1/-/gl/0001833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
Connections:
- net 3V3: now also SW1.3
- net at ESP32_NODEMCU1.10 (D27), R3.1, SW1.2 (K): now also SW1.4
Other:
- note added: "Note:"
- note removed: "Note: custom_push footprint not correct!"
Changed lines of the file:
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@@
 		)
 	)
-	(text "Note: \ncustom_push footprint not correct!"
+	(text "Note: \n\n"
 		(exclude_from_sim no)
 		(at 14.986 17.018 0)
@@
 			)
 		)
-		(property "Footprint" "Button_Switch_SMD:SW_Push_1P1T_NO_CK_KMR2"
+		(property "Footprint" "_myLibrary:button_push_sms"
 			(at 91.44 88.9 0)
 			(effects
@@
 			)
 		)
-		(property "Datasheet" "http://www.apem.com/int/index.php?controller=attachment&id_attachment=1371"
+		(property "Datasheet" "https://asset.conrad.com/media10/add/160267/c1/-/gl/000183373DS01/datenblatt-183373-mentor-12541004-12541004-drucktaster-12-v-dcac-005-a-1-x-ausein-tastend-1-st.pdf"
 			(at 91.44 88.9 0)
 			(effects
@@
 			)
 		)
-		(property "Description" "MEC 5E single pole normally-open tactile switch"
+		(property "Description" "https://www.conrad.at/de/p/mentor-1254-1004-1254-1004-drucktaster-12-v-dc-ac-0-05-a-1-x-aus-ein-tastend-1-st-183373.html"
 			(at 83.82 88.9 0)
 			(effects
@@
 			)
 		)
+		(property "Field5" "https://asset.conrad.com/media10/add/160267/c1/-/gl/000183373DS01/datenblatt-183373-mentor-12541004-12541004-drucktaster-12-v-dcac-005-a-1-x-ausein-tastend-1-st.pdf"
+			(at 83.82 88.9 90)
+			(effects
+				(font
+					(size 1.27 1.27)
+				)
+				(hide yes)
+			)
+		)
 		(pin "2"
 		)
 		(pin "1"
 		)
-		(pin "1"
-		)
-		(pin "2"
+		(pin "3"
+		)
+		(pin "4"
 		)
 		(instances
